Commit message: update parkour_quadruped.urdf

File: resources/robots/parkour_quadruped/urdf/parkour_quadruped.urdf (robot description, URDF)
Before this commit: robot Lite3_Simplified_Visual, 17 links, 16 joints
Links:
- link FL_SHANK: geometry collision cylinder length=0.10 radius=0.015; collision cylinder length=0.12 radius=0.015
- link FL_THIGH: geometry collision box size=0.04 0.045 0.20; visual cylinder length=0.20 radius=0.022
- link FR_SHANK: geometry collision cylinder length=0.10 radius=0.015; collision cylinder length=0.12 radius=0.015
- link FR_THIGH: geometry collision box size=0.04 0.045 0.20; visual cylinder length=0.20 radius=0.022
- link HL_SHANK: geometry collision cylinder length=0.10 radius=0.015; collision cylinder length=0.12 radius=0.015
- link HL_THIGH: geometry collision box size=0.04 0.045 0.20; visual cylinder length=0.20 radius=0.022
- link HR_SHANK: geometry collision cylinder length=0.10 radius=0.015; collision cylinder length=0.12 radius=0.015
- link HR_THIGH: geometry collision box size=0.04 0.045 0.20; visual cylinder length=0.20 radius=0.022
- link TORSO: geometry collision box size=0.25 0.20 0.12; collision box size=0.50 0.10 0.12
Joints:
- joint FL_HipX_joint: origin xyz=0.1745 0.11 0 -> xyz=0.1745 0.062 0
- joint FL_HipY_joint: origin xyz=0 0 0 -> xyz=0 0.09735 0
- joint FL_Knee_joint: origin xyz=0 0 -0.18 -> xyz=0 0 -0.20
- joint FR_HipX_joint: origin xyz=0.1745 -0.11 0 -> xyz=0.1745 -0.062 0
- joint FR_HipY_joint: origin xyz=0 0 0 -> xyz=0 -0.09735 0
- joint FR_Knee_joint: origin xyz=0 0 -0.18 -> xyz=0 0 -0.20
- joint HL_HipX_joint: origin xyz=-0.1745 0.11 0 -> xyz=-0.1745 0.062 0
- joint HL_HipY_joint: origin xyz=0 0 0 -> xyz=0 0.09735 0
- joint HL_Knee_joint: origin xyz=0 0 -0.18 -> xyz=0 0 -0.20
- joint HR_HipX_joint: origin xyz=-0.1745 -0.11 0 -> xyz=-0.1745 -0.062 0
- joint HR_HipY_joint: origin xyz=0 0 0 -> xyz=0 -0.09735 0
- joint HR_Knee_joint: origin xyz=0 0 -0.18 -> xyz=0 0 -0.20
